File: electronics/ofen.sch (KiCad schematic (older format))
At the start: 54 parts, among them J1 motor, J2 DC, J3 AC, J4 AC, J5 AC, Q1 Q_NPN_CBE, Q2 Q_NPN_CBE, Q3 Q_NPN_CBE, Q4 Q_NPN_CBE, Q5 BTA16-600B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

Commit message: made a PCB
Parts:
- removed C2, C3, C4, C5: 1µ, Capacitor_THT:CP_Radial_D6.3mm_P2.50mm, symbol Device:CP
- removed J3, J4, J5: AC, TerminalBlock:TerminalBlock_Altech_AK300-3_P5.00mm, symbol Connector_Generic:Conn_01x02
- added C2, C3, C4: 22n, Capacitor_THT:C_Disc_D4.3mm_W1.9mm_P5.00mm, symbol Device:C
- added J3, J4: Screw_Terminal_01x03, TerminalBlock:TerminalBlock_Altech_AK300-3_P5.00mm, symbol Connector:Screw_Terminal_01x03
- C5: renamed from C?; value 460n -> 470n; footprint (none) -> Capacitor_THT:C_Rect_L7.0mm_W4.5mm_P5.00mm
- C7, C8: renamed from C?; footprint (none) -> Capacitor_THT:C_Rect_L7.0mm_W4.5mm_P5.00mm
- Q5: footprint Package_TO_SOT_THT:TO-220-3_Horizontal_TabUp -> Connector_Wire:SolderWire-0.75sqmm_1x03_P4.8mm_D1.25mm_OD2.3mm
- gave numbers to parts that had none: 1
Connections:
- net GND: now also C2.1, C3.1, C4.1
- net at U1.10 (D19): now also SW3.1, C3.2
- net at U1.11 (D21): now also SW4.1, C4.2
- net at U1.23 (D25): no longer SW4.1
- net at U1.24 (D26): no longer SW3.1
- net at U1.25 (D27): no longer SW2.1
- net at U1.27 (D12): now also R13.2; no longer SW1.1 (A)
- net at U1.28 (D13): now also SW1.1 (A); no longer R13.2
- net at U1.9 (D18): now also SW2.1, C2.2
- net at T1.1 (AA), T2.1 (AA): now also J4.1 (Pin_1), J4.2 (Pin_2), J4.3 (Pin_3)
- net at T2.2 (AB): now also R20.2; no longer R20.1
- net at C6.2, Q5.1 (A1), R17.1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: now also R20.1; no longer R20.2
- net at Q5.2 (A2), R15.1, R18.1: now also J3.1 (Pin_1), J3.2 (Pin_2), J3.3 (Pin_3)
Other:
- moved on the sheet: SW1, SW2, SW3, SW4

Commit message: added resistor in parallel to the thermocouple to prevent OpAmp from destroying the ESP32
Parts:
- added R26: 15k, Resistor_THT:R_Axial_DIN0207_L6.3mm_D2.5mm_P10.16mm_Horizontal, symbol Device:R
Connections:
- net at R14.1, R16.2, U3.2 (-): now also R26.1
- net at TC1.1 (+), U3.3 (+): now also R26.2
- no-connect marks 0 -> 12
Changed lines of the file:
@@
 	6700 4900 6800 4900
 Wire Wire Line
-	7500 5000 7500 5600
+	7500 5000 7500 5300
 Wire Wire Line
 	7500 5700 7500 5600
@@
 	7700 5000 7800 5000
 Wire Wire Line
-	7800 4800 7400 4800
+	7800 4800 7600 4800
 Wire Wire Line
 	6700 3400 5700 3400
@@
 Wire Wire Line
 	6200 2600 5700 2600
+$Comp
+L Device:R R26
+U 1 1 60135609
+P 7600 5050
+F 0 "R26" H 7700 4900 50  0000 R CNN
+F 1 "15k" V 7600 5125 50  0000 R CNN
+F 2 "Resistor_THT:R_Axial_DIN0207_L6.3mm_D2.5mm_P10.16mm_Horizontal" V 7530 5050 50  0001 C CNN
+F 3 "~" H 7600 5050 50  0001 C CNN
+	1    7600 5050
+	1    0    0    1
+$EndComp
+Wire Wire Line
+	7600 4900 7600 4800
+Connection ~ 7600 4800
+Wire Wire Line
+	7600 4800 7400 4800
+Wire Wire Line
+	7600 5200 7600 5300
+Wire Wire Line
+	7600 5300 7500 5300
+Connection ~ 7500 5300
+Wire Wire Line
+	7500 5300 7500 5600
+NoConn ~ 5700 2700
+NoConn ~ 5700 2800
+NoConn ~ 5700 2900
+NoConn ~ 5700 3000
+NoConn ~ 4700 2500
+NoConn ~ 4700 2600
+NoConn ~ 4700 2700
+NoConn ~ 4700 2800
+NoConn ~ 4700 2900
+NoConn ~ 4700 3000
+NoConn ~ 4700 3400
+NoConn ~ 4700 3500
 $EndSCHEMATC

Commit message: added opamp offset trimmer to schematic and pcb
Parts:
- removed J4: Screw_Terminal_01x03, TerminalBlock:TerminalBlock_Altech_AK300-3_P5.00mm, symbol Connector:Screw_Terminal_01x03
- removed U3: LMH6609MA, Package_DIP:DIP-8_W7.62mm_LongPads, symbol Amplifier_Operational:LMH6609MA
- added J4, J5: AC_OUT, Connector_Wire:SolderWire-0.75sqmm_1x02_P4.8mm_D1.25mm_OD2.3mm, symbol Connector_Generic:Conn_01x02
- added RV1: 10k, Connector_PinHeader_2.54mm:PinHeader_1x03_P2.54mm_Vertical, symbol Device:R_POT_TRIM
- added U3: LM6361, Package_DIP:DIP-8_W7.62mm_Socket_LongPads, symbol Amplifier_Operational:LM6361
- J3: value Screw_Terminal_01x03 -> AC_IN
- U1: symbol Custom:ESP32 -> ofen-rescue:ESP32-Custom
Connections:
- net +5V: now also RV1.2, U3.7 (V+)
- net -5V: now also U3.4 (V-)
- net GND: now also J3.2 (Pin_2), U1.23 (D25), U1.24 (D26), U1.25 (D27), U1.26 (D14), U1.3 (D15), U1.4 (D2), U1.5 (D4)
- net at R14.2, U1.19 (D34): now also U3.6
- net at T1.1 (AA), T2.1 (AA): now also J3.1 (Pin_1), J5.1 (Pin_1), J5.2 (Pin_2)
- net at R14.1, R16.2, R26.1: now also U3.2 (-)
- net at R26.2, TC1.1 (+): now also U3.3 (+)
- net at J3.3 (Pin_3), Q5.2 (A2), R15.1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: now also J4.1 (Pin_1), J4.2 (Pin_2); no longer J3.1 (Pin_1), J3.2 (Pin_2)
- new net: RV1.3, U3.1 (VOS)
- new net: RV1.1, U3.8 (VOS)
- no-connect marks 12 -> 2
Other:
- moved on the sheet: J3
Changed lines of the file:
@@
 $EndDescr
-$Comp
-L Custom:ESP32 U1
-U 1 1 5FF1B380
-P 5200 3000
-F 0 "U1" H 5200 3965 50  0000 C CNN
-F 1 "ESP32" H 5200 3874 50  0000 C CNN
-F 2 "custom:ESP32-DevModule" H 5200 3100 50  0001 C CNN
-F 3 "" H 5200 3100 50  0001 C CNN
-	1    5200 3000
-	1    0    0    -1
-$EndComp
 $Comp
 L Device:Q_NPN_CBE Q1
@@
 $EndComp
 Wire Wire Line
-	4500 2400 4700 2400
-Wire Wire Line
 	4500 2400 4500 2500
 $Comp
@@
 	4200 1800 4200 1900
 $Comp
-L Amplifier_Operational:LMH6609MA U3
-U 1 1 6014CFCF
-P 7100 4900
-F 0 "U3" H 7444 4946 50  0000 L CNN
-F 1 "LMH6609MA" H 7444 4855 50  0000 L CNN
-F 2 "Package_DIP:DIP-8_W7.62mm_LongPads" H 7000 4700 50  0001 L CNN
-F 3 "http://www.ti.com/lit/ds/symlink/lmh6609.pdf" H 7250 5050 50  0001 C CNN
-	1    7100 4900
-	-1   0    0    -1
-$EndComp
-$Comp
 L Device:R R14
 U 1 1 6015686F
@@
 L power:+5V #PWR013
 U 1 1 60167835
-P 7200 4500
-F 0 "#PWR013" H 7200 4350 50  0001 C CNN
-F 1 "+5V" H 7215 4673 50  0000 C CNN
-F 2 "" H 7200 4500 50  0001 C CNN
-F 3 "" H 7200 4500 50  0001 C CNN
-	1    7200 4500
+P 7200 4400
+F 0 "#PWR013" H 7200 4250 50  0001 C CNN
+F 1 "+5V" H 7215 4573 50  0000 C CNN
+F 2 "" H 7200 4400 50  0001 C CNN
+F 3 "" H 7200 4400 50  0001 C CNN
+	1    7200 4400
 	-1   0    0    -1
 $EndComp
@@
 	8600 1100 8600 1300
 Wire Wire Line
-	4700 2400 5700 2400
-Connection ~ 4700 2400
-Wire Wire Line
 	6200 1200 6200 1100
 Wire Wire Line
@@
 	-1   0    0    -1
 $EndComp
-Wire Wire Line
-	9500 1200 9500 1600
 Connection ~ 9500 1600
 $Comp
@@
 	4700 3200 4600 3200
 Wire Wire Line
-	4600 3200 4600 2900
-Wire Wire Line
-	4600 2900 3400 2900
-Wire Wire Line
-	3400 2900 3400 1400
-Wire Wire Line
 	3400 1400 2200 1400
 Connection ~ 2200 1400
@@
 	4700 3100 4650 3100
 Wire Wire Line
-	4650 3100 4650 2800
-Wire Wire Line
-	4650 2800 3500 2800
-Wire Wire Line
-	3500 2800 3500 1300
-Wire Wire Line
 	3500 1300 1800 1300
 Connection ~ 1800 1300
@@
 L Connector:Screw_Terminal_01x03 J3
 U 1 1 602C6C50
-P 9800 700
-F 0 "J3" H 9880 742 50  0000 L CNN
-F 1 "Screw_Terminal_01x03" H 9880 651 50  0000 L CNN
-F 2 "TerminalBlock:TerminalBlock_Altech_AK300-3_P5.00mm" H 9800 700 50  0001 C CNN
-F 3 "~" H 9800 700 50  0001 C CNN
-	1    9800 700
-	1    0    0    -1
-$EndComp
-$Comp
-L Connector:Screw_Terminal_01x03 J4
-U 1 1 602D5E02
-P 9800 1100
-F 0 "J4" H 9880 1142 50  0000 L CNN
-F 1 "Screw_Terminal_01x03" H 9880 1051 50  0000 L CNN
-F 2 "TerminalBlock:TerminalBlock_Altech_AK300-3_P5.00mm" H 9800 1100 50  0001 C CNN
-F 3 "~" H 9800 1100 50  0001 C CNN
-	1    9800 1100
-	1    0    0    -1
-$EndComp
-Wire Wire Line
-	9500 1200 9600 1200
-Wire Wire Line
-	9600 1200 9600 1100
-Connection ~ 9600 1200
-Wire Wire Line
-	9600 1100 9600 1000
-Connection ~ 9600 1100
-Wire Wire Line
-	8000 800  9600 800
-Wire Wire Line
-	9600 700  9600 800
-Connection ~ 9600 800
-Wire Wire Line
-	9600 700  9600 600
-Connection ~ 9600 700
+P 9800 900
+F 0 "J3" H 9880 942 50  0000 L CNN
+F 1 "AC_IN" H 9880 851 50  0000 L CNN
+F 2 "TerminalBlock:TerminalBlock_Altech_AK300-3_P5.00mm" H 9800 900 50  0001 C CNN
+F 3 "~" H 9800 900 50  0001 C CNN
+	1    9800 900
+	1    0    0    1
+$EndComp
+Wire Wire Line
+	8000 800  8700 800
 Wire Wire Line
 	7000 2500 7000 2600
@@
 Wire Wire Line
 	7500 5300 7500 5600
-NoConn ~ 5700 2700
-NoConn ~ 5700 2800
-NoConn ~ 5700 2900
-NoConn ~ 5700 3000
-NoConn ~ 4700 2500
-NoConn ~ 4700 2600
-NoConn ~ 4700 2700
-NoConn ~ 4700 2800
-NoConn ~ 4700 2900
-NoConn ~ 4700 3000
 NoConn ~ 4700 3400
 NoConn ~ 4700 3500
+$Comp
+L Amplifier_Operational:LM6361 U3
+U 1 1 6023E246
+P 7100 4900
+F 0 "U3" H 7150 5150 50  0000 C CNN
+F 1 "LM6361" H 7250 5050 50  0000 C CNN
+F 2 "Package_DIP:DIP-8_W7.62mm_Socket_LongPads" H 7150 5100 50  0001 C CNN
+F 3 "http://www.ti.com/lit/ds/symlink/lm6161.pdf" H 7250 5200 50  0001 C CNN
+	1    7100 4900
+	-1   0    0    -1
+$EndComp
+$Comp
+L Device:R_POT_TRIM RV1
+U 1 1 60241F8D
+P 6700 5950
+F 0 "RV1" H 6600 5900 50  0000 R CNN
+F 1 "10k" H 6600 6000 50  0000 R CNN
+F 2 "Connector_PinHeader_2.54mm:PinHeader_1x03_P2.54mm_Vertical" H 6700 5950 50  0001 C CNN
+F 3 "~" H 6700 5950 50  0001 C CNN
+	1    6700 5950
+	-1   0    0    1
+$EndComp
+Wire Wire Line
+	7000 5200 7000 5700
+Wire Wire Line
+	7000 5700 6700 5700
+Wire Wire Line
+	6700 5700 6700 5800
+Wire Wire Line
+	6700 6100 6700 6200
+Wire Wire Line
+	6700 6200 7100 6200
+Wire Wire Line
+	7100 6200 7100 5200
+Wire Wire Line
+	6550 5950 6450 5950
+Wire Wire Line
+	6450 5950 6450 4500
+Wire Wire Line
+	6450 4500 7200 4500
+Connection ~ 7200 4500
+Wire Wire Line
+	7200 4500 7200 4400
+Wire Wire Line
+	9500 1000 9600 1000
+Wire Wire Line
+	9500 1000 9500 1200
+$Comp
+L power:GND #PWR025
+U 1 1 6032D73A
+P 9300 1000
+F 0 "#PWR025" H 9300 750 50  0001 C CNN
+F 1 "GND" H 9305 827 50  0000 C CNN
+F 2 "" H 9300 1000 50  0001 C CNN
+F 3 "" H 9300 1000 50  0001 C CNN
+	1    9300 1000
+	1    0    0    -1
+$EndComp
+Wire Wire Line
+	9300 1000 9300 900
+Wire Wire Line
+	4700 2400 5700 2400
+Wire Wire Line
+	4500 2400 4700 2400
+Connection ~ 4700 2400
+Wire Wire Line
+	5700 2700 5700 2800
+Connection ~ 5700 2800
+Wire Wire Line
+	5700 2800 5700 2900
+Connection ~ 5700 2900
+Wire Wire Line
+	5700 2900 5700 3000
+$Comp
+L power:GND #PWR016
+U 1 1 6034FD19
+P 5900 2800
+F 0 "#PWR016" H 5900 2550 50  0001 C CNN
+F 1 "GND" H 5905 2627 50  0000 C CNN
+F 2 "" H 5900 2800 50  0001 C CNN
+F 3 "" H 5900 2800 50  0001 C CNN
+	1    5900 2800
+	1    0    0    -1
+$EndComp
+Wire Wire Line
+	5900 2800 5900 2700
+Wire Wire Line
+	5900 2700 5700 2700
+Connection ~ 5700 2700
+Wire Wire Line
+	3500 2800 3500 1300
+Wire Wire Line
+	3400 2900 3400 1400
+$Comp
+L ofen-rescue:ESP32-Custom U1
+U 1 1 5FF1B380
+P 5200 3000
+F 0 "U1" H 5200 3965 50  0000 C CNN
+F 1 "ESP32" H 5200 3874 50  0000 C CNN
+F 2 "custom:ESP32-DevModule" H 5200 3100 50  0001 C CNN
+F 3 "" H 5200 3100 50  0001 C CNN
+	1    5200 3000
+	1    0    0    -1
+$EndComp
+Wire Wire Line
+	4650 2800 3500 2800
+Wire Wire Line
+	4650 3100 4650 2800
+Wire Wire Line
+	4600 2900 3400 2900
+Wire Wire Line
+	4600 3200 4600 2900
+Wire Wire Line
+	4700 2400 4700 2500
+Connection ~ 4700 2500
+Wire Wire Line
+	4700 2500 4700 2600
+Connection ~ 4700 2600
+Wire Wire Line
+	4700 2600 4700 2700
+$Comp
+L Connector_Generic:Conn_01x02 J5
+U 1 1 6038E74D
+P 9800 1200
+F 0 "J5" H 9880 1192 50  0000 L CNN
+F 1 "AC_OUT" H 9880 1101 50  0000 L CNN
+F 2 "Connector_Wire:SolderWire-0.75sqmm_1x02_P4.8mm_D1.25mm_OD2.3mm" H 9800 1200 50  0001 C CNN
+F 3 "~" H 9800 1200 50  0001 C CNN
+	1    9800 1200
+	1    0    0    -1
+$EndComp
+$Comp
+L Connector_Generic:Conn_01x02 J4
+U 1 1 60390C15
+P 8900 1100
+F 0 "J4" H 8980 1092 50  0000 L CNN
+F 1 "AC_OUT" H 8980 1001 50  0000 L CNN
+F 2 "Connector_Wire:SolderWire-0.75sqmm_1x02_P4.8mm_D1.25mm_OD2.3mm" H 8900 1100 50  0001 C CNN
+F 3 "~" H 8900 1100 50  0001 C CNN
+	1    8900 1100
+	1    0    0    -1
+$EndComp
+Wire Wire Line
+	8700 1200 8700 1100
+Wire Wire Line
+	8700 1100 8700 800
+Connection ~ 8700 1100
+Wire Wire Line
+	9600 1300 9500 1300
+Connection ~ 9500 1300
+Wire Wire Line
+	9500 1300 9500 1600
+Wire Wire Line
+	9600 1200 9500 1200
+Connection ~ 9500 1200
+Wire Wire Line
+	9500 1200 9500 1300
+Wire Wire Line
+	9300 900  9600 900
+Wire Wire Line
+	9600 800  8700 800
+Connection ~ 8700 800
 $EndSCHEMATC
