File: electronics/ofen.sch (KiCad schematic (older format))
At the start: 53 parts, among them J1 motor, J2 DC, J3 Screw_Terminal_01x03, J4 Screw_Terminal_01x03, Q1 Q_NPN_CBE, Q2 Q_NPN_CBE, Q3 Q_NPN_CBE, Q4 Q_NPN_CBE, Q5 BTA16-600B, SW1 SW_SPST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

Commit message: redid adc calibration and some small changes
Parts:
- U1: symbol Custom:ESP32 -> ofen-rescue:ESP32-Custom
Changed lines of the file:
@@
 $EndDescr
 $Comp
-L Custom:ESP32 U1
+L ofen-rescue:ESP32-Custom U1
 U 1 1 5FF1B380
 P 5200 3000
